File: Eagle/UwU Bot.brd (EAGLE design)
At the start: 100 x 80 mm, 8 parts, among them U1 173010535

Commit message: updated Eagle
Parts:
- moved MOTOR2 143.4 mm to (67.3, 63.5), turned to 270 degrees
- moved MOTOR1 142.7 mm to (67.3, 36.8), turned to 270 degrees
- moved U1 125.8 mm to (49.5, 10.2), turned to 90 degrees
- moved DISPLAY_CON 122.2 mm to (24.1, 8.89)
- moved STEPPER_MOTOR_DRIVER1 111.2 mm to (53.3, 36.8)
- moved STEPPER_MOTOR_DRIVER2 110.8 mm to (53.3, 63.5)
- moved ESP32 54.6 mm to (24.1, 47.0), turned to 180 degrees
- moved U$1 44.4 mm to (59.7, 16.5), turned to 270 degrees
Connections:
- net N$1 renamed GND3
- net N$7 renamed GND2
- removed net 12V: STEPPER_MOTOR_DRIVER1.16, STEPPER_MOTOR_DRIVER2.16
- removed net N$10: U$1.P$3
- removed net N$11: U$1.P$4
- removed net N$14: ESP32.33
- removed net N$15: ESP32.34
- removed net N$17: ESP32.36
- removed net N$18: ESP32.37
- removed net N$19: ESP32.38
- removed net N$21: ESP32.2
- removed net N$22: ESP32.3
- removed net N$23: ESP32.4
- removed net N$24: MOTOR2.4, STEPPER_MOTOR_DRIVER2.12
- removed net N$25: MOTOR2.3, STEPPER_MOTOR_DRIVER2.11
- removed net N$30: MOTOR1.3, STEPPER_MOTOR_DRIVER1.11
- removed net N$31: MOTOR1.4, STEPPER_MOTOR_DRIVER1.12
- removed net N$32: U1.1
- removed net N$35: ESP32.16
- removed net N$36: ESP32.17
- removed net N$37: ESP32.18
- removed net N$5: ESP32.24
- new net 1A: MOTOR1.3, STEPPER_MOTOR_DRIVER1.12
- new net 1A#2: MOTOR2.3, STEPPER_MOTOR_DRIVER2.12
- new net N$1: MOTOR1.4, STEPPER_MOTOR_DRIVER1.11
- new net VIN: STEPPER_MOTOR_DRIVER1.16, STEPPER_MOTOR_DRIVER2.16, U$1.P$3, U$1.P$4, U1.1
- net N$4: now also MOTOR2.4, STEPPER_MOTOR_DRIVER2.11; no longer ESP32.23
Routing:
- net GND: track 0.00 -> 188.8 mm, vias 0 -> 1
- net IO5: track 0.00 -> 118.1 mm, vias 0 -> 3
- net IO19: track 0.00 -> 115.9 mm, vias 0 -> 1
- net VIN: track 0.00 -> 111.3 mm
- net IO4: track 0.00 -> 110.7 mm, vias 0 -> 1
- net VOUT: track 0.00 -> 90.4 mm, vias 0 -> 1
- net 3V3: track 0.00 -> 75.9 mm, vias 0 -> 1
- net IO12: track 0.00 -> 74.2 mm
- net IO16: track 0.00 -> 67.8 mm, vias 0 -> 2
- net IO15: track 0.00 -> 63.0 mm
- net IO26: track 0.00 -> 61.7 mm
- net IO18: track 0.00 -> 55.4 mm
- net IO22: track 0.00 -> 53.9 mm
- net IO32: track 0.00 -> 53.5 mm, vias 0 -> 1
- net IO17: track 0.00 -> 48.2 mm
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Other:
- board size 100 x 80 mm -> 77.1 x 80 mm
