File: Eagle/UwU Bot.sch (EAGLE design)
At the start: 8 parts, among them U1 173010535

Commit message: updated Eagle
Connections:
- removed net 12V: STEPPER_MOTOR_DRIVER1.VMOT, STEPPER_MOTOR_DRIVER2.VMOT
- removed net N$10: U$1.P$3
- removed net N$11: U$1.P$4
- removed net N$14: ESP32.IO0
- removed net N$15: ESP32.IO2
- removed net N$17: ESP32.SD1
- removed net N$18: ESP32.SD0
- removed net N$19: ESP32.CLK
- removed net N$21: ESP32.EN
- removed net N$22: ESP32.SENSOR_VP
- removed net N$23: ESP32.SENSOR_VN
- removed net N$24: MOTOR2.4, STEPPER_MOTOR_DRIVER2.1A
- removed net N$25: MOTOR2.3, STEPPER_MOTOR_DRIVER2.1B
- removed net N$30: MOTOR1.3, STEPPER_MOTOR_DRIVER1.1B
- removed net N$31: MOTOR1.4, STEPPER_MOTOR_DRIVER1.1A
- removed net N$32: U1.VIN
- removed net N$35: ESP32.SD2
- removed net N$36: ESP32.SD3
- removed net N$37: ESP32.CMD
- removed net N$5: ESP32.RXD0
- removed net N$7: ESP32.GND2
- new net 1A: MOTOR1.3, STEPPER_MOTOR_DRIVER1.1A
- new net 1A#2: MOTOR2.3, STEPPER_MOTOR_DRIVER2.1A
- new net VIN: STEPPER_MOTOR_DRIVER1.VMOT, STEPPER_MOTOR_DRIVER2.VMOT, U$1.P$3, U$1.P$4, U1.VIN
- net N$1: now also MOTOR1.4, STEPPER_MOTOR_DRIVER1.1B; no longer ESP32.GND3
- net N$4: now also MOTOR2.4, STEPPER_MOTOR_DRIVER2.1B; no longer ESP32.TXD0
